Commit message: feat: add initial Active Vision Platform project

File: Active Vision Platform/urdf/Active Vision Platform.urdf (robot description, URDF)
Before this commit: robot 主动视觉云台001.SLDASM, 3 links, 2 joints
Links:
- link Empty_Link1: geometry collision mesh filename=package://Active Vision Platform/meshes/Empty_Link1.STL; visual mesh filename=package://Active Vision Platform/meshes/Empty_Link1.STL
- link Empty_Link2: geometry collision mesh filename=package://Active Vision Platform/meshes/Empty_Link2.STL; visual mesh filename=package://Active Vision Platform/meshes/Empty_Link2.STL
- link base_link: geometry collision mesh filename=package://Active Vision Platform/meshes/base_link.STL; visual mesh filename=package://Active Vision Platform/meshes/base_link.STL

File: Active_Vision_Platform/urdf/Active_Vision_Platform.urdf (robot description, URDF)
Before this commit: robot 主动视觉云台001.SLDASM, 3 links, 2 joints
Links:
- link Empty_Link1: geometry collision mesh filename=./meshes/Empty_Link1.STL; visual mesh filename=./meshes/Empty_Link1.STL
- link Empty_Link2: geometry collision mesh filename=./meshes/Empty_Link2.STL; visual mesh filename=./meshes/Empty_Link2.STL
- link base_link: geometry collision mesh filename=./meshes/base_link.STL; visual mesh filename=./meshes/base_link.STL
